Commit message: [ktsui] correcting maki.urdf. 1) change 'swivel' to 'pan'. 2) change eye/eyelid/iris 1 to _right. 3) change eye/eyelid/iris 2 to _left.

File: maki.urdf (robot description, URDF)
Before this commit: robot maki, 11 links, 10 joints
Links:
- removed link eye1
- removed link eye2
- removed link eyelid1
- removed link eyelid2
- removed link iris1
- removed link iris2
- removed link virtual_eye2
- added link eye_left; visual sphere radius=0.15
- added link eye_right; visual sphere radius=0.15
- added link eyelid_left; visual box size=0.3 0.05 0.05
- added link eyelid_right; visual box size=0.3 0.05 0.05
- added link iris_left; visual sphere radius=0.05
- added link iris_right; visual sphere radius=0.05
- added link virtual_eye_left
Joints:
- removed joint eye1_swivel
- removed joint eye1_tilt
- removed joint eye2_swivel
- removed joint eye2_tilt
- removed joint eyelid1_joint
- removed joint eyelid2_joint
- removed joint head_swivel
- removed joint iris1_joint
- removed joint iris2_joint
- added joint eye_left_pan: type continuous, parent head, child virtual_eye_left, origin xyz=0.4 0.25 0.25, axis 0 0 1, mimic joint=eye_right_pan
- added joint eye_left_tilt: type continuous, parent virtual_eye_left, child eye_left, axis 0 1 0, mimic joint=eye_right_tilt
- added joint eye_right_pan: type revolute, parent head, child virtual_eye, origin xyz=0.4 -0.25 0.25, axis 0 0 1, limit lower=-0.337 upper=0.266 effort=1000.0 velocity=0.5
- added joint eye_right_tilt: type revolute, parent virtual_eye, child eye_right, axis 0 1 0, limit lower=-0.501 upper=0.445 effort=1000.0 velocity=0.5
- added joint eyelid_left_joint: type continuous, parent head, child eyelid_left, origin xyz=0.4 0.25 0.25, axis 0 1 0, mimic joint=eyelid_right_joint
- added joint eyelid_right_joint: type revolute, parent head, child eyelid_right, origin xyz=0.4 -0.25 0.25, axis 0 1 0, limit lower=-0.179 upper=0.712 effort=1000.0 velocity=0.5
- added joint head_pan: type revolute, parent base_link, child virtual_head, origin xyz=0 0 0, axis 0 0 1, limit lower=-1.309 upper=1.308 effort=1000.0 velocity=0.5
- added joint iris_left_joint: type fixed, parent eye_left, child iris_left, origin xyz=0.12 0 0
- added joint iris_right_joint: type fixed, parent eye_right, child iris_right, origin xyz=0.12 0 0

Commit message: [ktsui] prior maki.urdf was NOT to scale. rework dimensions and placements to better approximate actual dimensions of MAKIv1.4. Changed iris to cylinder and added cylindrical pupil. Added placement for webcam (in mouth)

File: maki.urdf (robot description, URDF)
Before this commit: robot maki, 11 links, 10 joints
Links:
- removed link virtual_eye
- added link mouth_camera; visual cylinder length=0.001 radius=0.001425
- added link pupil_left; visual cylinder length=0.005 radius=0.00633
- added link pupil_right; visual cylinder length=0.005 radius=0.00633
- added link virtual_eye_right
- link base_link: geometry visual cylinder length=0.16142 radius=0.069915
- link eye_left: geometry visual sphere radius=0.02211
- link eye_right: geometry visual sphere radius=0.02211
- link eyelid_left: geometry visual box size=0.032 0.005 0.005
- link eyelid_right: geometry visual box size=0.032 0.005 0.005
- link head: geometry visual sphere radius=0.0821
- link iris_left: geometry visual cylinder length=0.005 radius=0.015
- link iris_right: geometry visual cylinder length=0.005 radius=0.015
Joints:
- added joint pupil_left_joint: type fixed, parent iris_left, child pupil_left, origin xyz=0.005 0 0
- added joint pupil_right_joint: type fixed, parent iris_right, child pupil_right, origin xyz=0.005 0 0
- added joint robot_mouth_camera: type fixed, parent head, child mouth_camera, origin xyz=0.07 0 -0.044
- joint eye_left_pan: origin xyz=0.4 0.25 0.25 -> xyz=0.07589 0.03771 0
- joint eye_right_pan: child virtual_eye -> virtual_eye_right; origin xyz=0.4 -0.25 0.25 -> xyz=0.07589 -0.03771 0
- joint eye_right_tilt: parent virtual_eye -> virtual_eye_right
- joint eyelid_left_joint: origin xyz=0.4 0.25 0.25 -> xyz=0.07589 0.03771 0
- joint eyelid_right_joint: origin xyz=0.4 -0.25 0.25 -> xyz=0.07589 -0.03771 0
- joint head_tilt: origin xyz=0 0 1.6 -> xyz=0 0 0.243242
- joint iris_left_joint: origin xyz=0.12 0 0 -> xyz=0.015 0 0
- joint iris_right_joint: origin xyz=0.12 0 0 -> xyz=0.015 0 0

Commit message: [ktsui] adjust joint limits in maki.urdf. TODO: fix MAKI-URDF-Interface to not assume ordering and number of joints to match headers. BUG: Currently, eyelid position does NOT publish to /maki_command

File: maki.urdf (robot description, URDF)
Before this commit: robot maki, 14 links, 13 joints
Joints:
- joint eye_right_pan: limit lower=-0.337 upper=0.266 effort=1000.0 velocity=0.5 -> lower=-0.25 upper=0.25 effort=1000.0 velocity=0.5
- joint eye_right_tilt: limit lower=-0.501 upper=0.445 effort=1000.0 velocity=0.5 -> lower=-0.65 upper=0.6 effort=1000.0 velocity=0.5
- joint eyelid_right_joint: limit lower=-0.179 upper=0.712 effort=1000.0 velocity=0.5 -> lower=-0.785 upper=2.355 effort=1000.0 velocity=0.5
- joint head_pan: limit lower=-1.309 upper=1.308 effort=1000.0 velocity=0.5 -> lower=-1.0 upper=1.0 effort=1000.0 velocity=0.5

Commit message: [ktsui] swap eye_right and eye_left such that eye_right now mimics eye_left. Modify eyelid geometry so that eyelid does not collide with eye, iris, or pupil

File: maki.urdf (robot description, URDF)
Before this commit: robot maki, 14 links, 13 joints
Joints:
- joint eye_left_pan: limit (none) -> lower=-0.25 upper=0.25 effort=1000.0 velocity=0.5; mimic joint=eye_right_pan -> (none); type continuous -> revolute
- joint eye_left_tilt: limit (none) -> lower=-0.65 upper=0.6 effort=1000.0 velocity=0.5; mimic joint=eye_right_tilt -> (none); type continuous -> revolute
- joint eye_right_pan: limit lower=-0.25 upper=0.25 effort=1000.0 velocity=0.5 -> (none); mimic (none) -> joint=eye_left_pan; type revolute -> continuous
- joint eye_right_tilt: limit lower=-0.65 upper=0.6 effort=1000.0 velocity=0.5 -> (none); mimic (none) -> joint=eye_left_tilt; type revolute -> continuous
- joint eyelid_left_joint: limit (none) -> lower=-0.3 upper=1.0 effort=1000.0 velocity=0.5; mimic joint=eyelid_right_joint -> (none); type continuous -> revolute
- joint eyelid_right_joint: limit lower=-0.785 upper=2.355 effort=1000.0 velocity=0.5 -> (none); mimic (none) -> joint=eyelid_left_joint; type revolute -> continuous

Commit message: [ktsui] begin fixing URDF joint limit positions to reflect actual servo positions

File: maki.urdf (robot description, URDF)
Before this commit: robot maki, 14 links, 13 joints
Links:
- removed link eye_left
- removed link eye_right
- removed link eyelid_left
- removed link eyelid_right
- removed link iris_left
- removed link iris_right
- removed link mouth_camera
- removed link pupil_left
- removed link pupil_right
- removed link virtual_eye_left
- removed link virtual_eye_right
- added link eye1; visual sphere radius=0.15
- added link eye2; visual sphere radius=0.15
- added link eyelid1; visual box size=0.3 0.05 0.05
- added link eyelid2; visual box size=0.3 0.05 0.05
- added link iris1; visual sphere radius=0.05
- added link iris2; visual sphere radius=0.05
- added link virtual_eye
- added link virtual_eye2
- link base_link: geometry visual cylinder length=1 radius=0.5
- link head: geometry visual sphere radius=0.6
Joints:
- removed joint eye_left_pan
- removed joint eye_left_tilt
- removed joint eye_right_pan
- removed joint eye_right_tilt
- removed joint eyelid_left_joint
- removed joint eyelid_right_joint
- removed joint head_pan
- removed joint iris_left_joint
- removed joint iris_right_joint
- removed joint pupil_left_joint
- removed joint pupil_right_joint
- removed joint robot_mouth_camera
- added joint eye1_swivel: type revolute, parent head, child virtual_eye, origin xyz=0.4 -0.25 0.25, axis 0 0 1, limit lower=-0.337 upper=0.266 effort=1000.0 velocity=0.5
- added joint eye1_tilt: type revolute, parent virtual_eye, child eye1, axis 0 1 0, limit lower=-0.501 upper=0.445 effort=1000.0 velocity=0.5
- added joint eye2_swivel: type continuous, parent head, child virtual_eye2, origin xyz=0.4 0.25 0.25, axis 0 0 1, mimic joint=eye1_swivel
- added joint eye2_tilt: type continuous, parent virtual_eye2, child eye2, axis 0 1 0, mimic joint=eye1_tilt
- added joint eyelid1_joint: type revolute, parent head, child eyelid1, origin xyz=0.4 -0.25 0.25, axis 0 1 0, limit lower=-0.179 upper=0.712 effort=1000.0 velocity=0.5
- added joint eyelid2_joint: type continuous, parent head, child eyelid2, origin xyz=0.4 0.25 0.25, axis 0 1 0, mimic joint=eyelid1_joint
- added joint head_swivel: type revolute, parent base_link, child virtual_head, origin xyz=0 0 0, axis 0 0 1, limit lower=-1.309 upper=1.308 effort=1000.0 velocity=0.5
- added joint iris1_joint: type fixed, parent eye1, child iris1, origin xyz=0.12 0 0
- added joint iris2_joint: type fixed, parent eye2, child iris2, origin xyz=0.12 0 0
- joint head_tilt: limit lower=-0.358 upper=0.394 effort=1000.0 velocity=0.5 -> lower=2.354 upper=2.764 effort=1000.0 velocity=0.5; origin xyz=0 0 0.243242 -> xyz=0 0 1.6 rpy=0 3.9 0
